Commit message: added random checkpoints

File: ws_tcc/install/tcc/share/tcc/urdf/robot.urdf (robot description, URDF)
Before this commit: robot limpeza, 6 links, 5 joints
Links:
- added link imu, mass 1e-5; collision box size=0.02 0.02 0.05; visual box size=0.02 0.02 0.05
Joints:
- added joint base_link_to_imu: type fixed, parent base_link, child imu, origin xyz=0.0 0.0 0.055 rpy=0 0 0
- joint base_link_to_front_wheel: axis 0 0 1 -> 0 1 0
- joint base_link_to_left_wheel: axis 0 0 1 -> 0 1 0; origin xyz=-0.048 -0.048 -0.1335 rpy=0 0 0 -> xyz=-0.048 0.048 -0.1335 rpy=0 0 0
- joint base_link_to_right_wheel: axis 0 0 1 -> 0 1 0; origin xyz=-0.048 0.048 -0.1335 rpy=0 0 0 -> xyz=-0.048 -0.048 -0.1335 rpy=0 0 0
